File: emg_amplifier.sch (KiCad schematic (older format))
At the start: 36 parts, among them J1 Conn_02x08_Row_Letter_Last, U1 OPA140DGK, U2 INA333AIDGKR, U3 OPA376xxD, U4 TLV9002IPWR

Commit message: Fixed naming and cleaned up libraries
Parts:
- U1: symbol alpha_parts:OPA140DGK -> FANTM_parts:OPA140DGK
Changed lines of the file:
@@
 INVERTING DUAL-SUPPLY TO \nSINGLE-SUPPLY AMPLIFIER CIRCUIT
 $Comp
-L alpha_parts:OPA140DGK U1
+L FANTM_parts:OPA140DGK U1
 U 1 1 60650A62
 P 1400 6900
+AR Path="/60650A62" Ref="U1"  Part="1"
+AR Path="/6043E029/60650A62" Ref="U1"  Part="1"
 F 0 "U1" H 1100 7150 50  0000 L CNN
 F 1 "OPA140DGK" H 1400 7050 50  0000 L CNN

Commit message: Adding the LP filter to the level shifter
Parts:
- removed R4: 3.9k, Resistor_SMD:R_0603_1608Metric, symbol Device:R_US
- removed R7: 33k, Resistor_SMD:R_0603_1608Metric, symbol Device:R_US
- removed R8: 2.7k, Resistor_SMD:R_0603_1608Metric, symbol Device:R_US
- added C?: 4700pF, Capacitor_SMD:C_0603_1608Metric, symbol Device:C
- added R?: 35.7k, Resistor_SMD:R_0603_1608Metric, symbol Device:R_US
- C5: value 43pF -> 4700pF; DK_Detail_Page https://www.digikey.com/en/products/detail/kemet/C0603C430J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 -> https://www.digikey.com/en/products/detail/tdk-corporation/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; Description CAP CER 43PF 50V C0G/NP0 0603 -> CAP CER 4700PF 50V C0G 0603; Digi-Key_PN 399-10050-1-ND -> 445-6912-1-ND; MPN C0603C430J5GACTU -> CGA3E2C0G1H472J080AA; Manufacturer KEMET -> TDK Corporation
- POT1: value TC33X-2-103E -> TC33X-2-102E; DK_Detail_Page /product-detail/en/bourns-inc/TC33X-2-103E/TC33X-103ETR-ND/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 -> https://www.digikey.com/en/products/detail/bourns-inc/TC33X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; Description TRIMMER 10K OHM 0.1W J LEAD TOP -> TRIMMER 1K OHM 0.1W J LEAD TOP; Digi-Key_PN TC33X-103ETR-ND -> TC33X-102ECT-ND; MPN TC33X-2-103E -> TC33X-2-102E
- R1: value 33k -> 36.5k; DK_Detail_Page https://www.digikey.com/en/products/detail/yageo/RC0603FR-0733KL/727159 -> https://www.digikey.com/en/products/detail/yageo/RC0603FR-0736K5L/727181; Description RES SMD 33K OHM 1% 1/10W 0603 -> (none); Digi-Key_PN 311-33.0KHRCT-ND -> (none); MPN RC0603FR-0733KL -> (none); Manufacturer Yageo -> (none); Tolerance ±1% -> (none)
Connections:
- net labels added: -4V5
- net labels removed: -5V
Other:
- note added: "INVERTING DUAL-SUPPLY TO \nSINGLE-SUPPLY AMPLIFIER CIRCUIT\n\nDesign referenced from \nTI's Analog Engineer's Circuit Cookbook: \nAmplifiers (Rev. A)\n\nPage 162\n"
- note removed: "INVERTING DUAL-SUPPLY TO \nSINGLE-SUPPLY AMPLIFIER CIRCUIT"
- moved on the sheet: C5, R1, R6

Commit message: Finalized rev dev.a.2 with improved filtering, power supply design, and silkscreen
Parts:
- removed C1, C4, C8: 0.1uF, Capacitor_SMD:C_0603_1608Metric, symbol Device:C
- removed C11: 0.033uF, Capacitor_SMD:C_0603_1608Metric, symbol Device:C
- removed C7, C9: 0.15uF, Capacitor_SMD:C_0603_1608Metric, symbol Device:C
- removed J1: Conn_02x08_Row_Letter_Last, Connector_PinHeader_2.54mm:PinHeader_2x08_P2.54mm_Vertical, symbol Connector_Generic:Conn_02x08_Odd_Even
- removed R10, R11, R12: 100k, Resistor_SMD:R_0603_1608Metric, symbol Device:R_US
- removed R13, R14, R15, R16, R17: 10k, Resistor_SMD:R_0603_1608Metric, symbol Device:R_US
- removed U4: TLV9002IPWR, Package_SO:TSSOP-8_4.4x3mm_P0.65mm, symbol Device:Opamp_Dual_Generic
- C10: value 0.15uF -> 0.1uF; DK_Detail_Page https://www.digikey.com/en/products/detail/samsung-electro-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 -> (none); Description CAP CER 0.15UF 16V X7R 0603 -> CAP CER 0.1UF 16V X7R 0603; Digi-Key Part Number 1276-1972-1-ND -> (none); Digi-Key_PN (none) -> 311-1088-1-ND; Digikey (none) -> https://www.digikey.com/en/products/detail/yageo/CC0603KRX7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; MPN (none) -> CC0603KRX7R7BB104; Manufacturer Samsung Electro-Mechanics -> Yageo; Manufacturer Product Number CL10B154KO8NNNC -> (none); Package 0603 -> (none); Package Size (none) -> 0603; Rated Voltage (none) -> 16V; Supplier (none) -> Yageo; Temperature (none) -> X7R; Voltage - Rated 16V -> (none)
- C11: renamed from C5; Temperature Coefficient (none) -> C0G
- C12, C13: value 0.033uF -> 0.1uF; DK_Detail_Page https://www.digikey.com/en/products/detail/yageo/CC0603KRX7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 -> (none); Description CAP CER 0.033UF 16V X7R 0603 -> CAP CER 0.1UF 16V X7R 0603; Digi-Key Part Number 311-4071-1-ND -> (none); Digi-Key_PN (none) -> 311-1088-1-ND; Digikey (none) -> https://www.digikey.com/en/products/detail/yageo/CC0603KRX7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; MPN (none) -> CC0603KRX7R7BB104; Manufacturer Product Number CC0603KRX7R7BB333 -> (none); Package 0603 -> (none); Package Size (none) -> 0603; Rated Voltage (none) -> 16V; Supplier (none) -> Yageo; Temperature (none) -> X7R; Voltage - Rated 16V -> (none)
- C6: Digi-Key_PN (none) -> 311-1088-1-ND; MPN (none) -> CC0603KRX7R7BB104; Manufacturer Product Number CC0603KRX7R7BB104 -> (none)
- C7: renamed from C2; Digi-Key_PN (none) -> 311-1088-1-ND; MPN (none) -> CC0603KRX7R7BB104; Manufacturer Product Number CC0603KRX7R7BB104 -> (none)
- C9: renamed from C?; Temperature Coefficient (none) -> C0G
- POT1: value TC33X-2-102E -> GAIN
- R5: renamed from R1; Description (none) -> RES SMD 36.5K OHM 1% 1/10W 0603; Digi-Key_PN (none) -> 311-36.5KHRCT-ND; MPN (none) -> RC0603FR-0736K5L; Tolerance (none) -> ±1%
- R9: renamed from R?; Description (none) -> RES 35.7K OHM 1% 1/10W 0603; Digi-Key_PN (none) -> RMCF0603FT35K7CT-ND; MPN (none) -> RMCF0603FT35K7; Manufacturer (none) -> Stackpole Electronics Inc; Package (none) -> 0603; Tolerance (none) -> ±1%
- renumbered C3 to C8, R9 to R10, R2 to R4, R3 to R6, R5 to R7, R6 to R8, U1 to U2, U2 to U3, U3 to U4
Connections:
- net labels removed: ACTIVE_HP_OUT, ACTIVE_LP_OUT, EMG_SHIFT, FIRST_ORDER_HP, FIRST_ORDER_LP, HP, HP_1, HP_2, HP_2_+, HP_2_MID, LP_1, LP_2, LP_2_+, LP_2_MID, PASSIVE_HP_OUT, PASSIVE_LP_OUT, RAW_EMG, SECOND_ORDER_HP, SECOND_ORDER_LP
- wire segments 181 -> 86
Other:
- note added: "Fc (-3dB) is 696.96Hz\nfor this low pass filter.\n"
- note added: "G = 1 + (100 kΩ / RG)\n"
- note removed: "1ST ORDER\nPASSIVE HP & LP FILTERS"
- note removed: "2ND ORDER\nACTIVE HP & LP FILTERS"
- note removed: "FILTER CONFIGURATION\n"
- note removed: "Fc = 1 / (2 * pi * R * C)\n= 1 / (2 * pi * 100kOhm * 0.15uF)\n= 10.61Hz\n"
- note removed: "Fc = 1 / (2 * pi * R * C)\n= 1 / (2 * pi * 10kOhm * 0.033uF) \n= 482.29Hz\n"
- note removed: "G = 1 + (100 kΩ / RG)\nG = 1 + (100 * 10^3 / 560)\nG = 179.57\n"

Commit message: Major overhaul given chip shortage. Completely redid the power supply, and refined the amps for the EMG to give better gain and use the full output range
Parts:
- removed C11, C9: 4700pF, Capacitor_SMD:C_0603_1608Metric, symbol Device:C
- removed R5: 36.5k, Resistor_SMD:R_0603_1608Metric, symbol Device:R_US
- removed U2: OPA140DGK, Package_SO:VSSOP-8_3.0x3.0mm_P0.65mm, symbol FANTM_parts:OPA140DGK
- removed U3: INA333AIDGKR, digikey-footprints:TSSOP-8_W3mm, symbol dk_Linear-Amplifiers-Instrumentation-OP-Amps-Buffer-Amps:INA333AIDGKR
- added C10, C8: 6800pF, Capacitor_SMD:C_0603_1608Metric, symbol Device:C
- added R2: 25.5k, Resistor_SMD:R_0603_1608Metric, symbol Device:R_US
- added TP2: RAW_EMG, digikey-footprints:Test_Point_D1.02mm, symbol dk_Test-Points:5011
- added U3: OPA375DCK, digikey-footprints:SC-70-5, symbol FANTM_parts:OPA375DCK
- added U4: INA818IDR, digikey-footprints:SOIC-8_W3.9mm, symbol FANTM_parts:INA818IDR
- C7: renamed from C8;  Temperature Coefficient X5R -> (none); Temperature Coefficient (none) -> X5R
- R5: renamed from R8; value 39k -> 46.4k; Description CRGCQ 0603 39K 1% -> RES SMD 46.4K OHM 1% 1/10W 0603; Digi-Key_PN A129707CT-ND -> 311-46.4KHRCT-ND; MPN CRGCQ0603F39K -> RC0603FR-0746K4L; Manufacturer TE Connectivity Passive Product -> Yageo
- renumbered C12 to C11, C13 to C12, C6 to C5, C7 to C6, C10 to C9, R4 to R1, R6 to R3, R7 to R4, R9 to R6, R10 to R7, U4 to U5
Connections:
- net labels added: -3V, BUFFER_FDBK, BUFFER_OUT, RG_1, RG_2, V_SHIFT
- net labels removed: -4V5
- wire segments 86 -> 88
Other:
- note added: "Fc (-3dB) is 611.84Hz\nfor this low pass filter.\n"
- note added: "G = 1 + (50 kΩ / RG)\n"
- note removed: "Fc (-3dB) is 696.96Hz\nfor this low pass filter.\n"
- note removed: "G = 1 + (100 kΩ / RG)\n"

Commit message: Finished rev dev.a.4 with safety improvements, better gain settings, and dc offset removal
Parts:
- removed C10, C8: 6800pF, Capacitor_SMD:C_0603_1608Metric, symbol Device:C
- removed R2: 25.5k, Resistor_SMD:R_0603_1608Metric, symbol Device:R_US
- removed R5: 46.4k, Resistor_SMD:R_0603_1608Metric, symbol Device:R_US
- removed U4: INA818IDR, digikey-footprints:SOIC-8_W3.9mm, symbol FANTM_parts:INA818IDR
- added C11, C12, C13: 4700pF, Capacitor_SMD:C_0603_1608Metric, symbol Device:C
- added C16, C17: 0.1uF, Capacitor_SMD:C_0603_1608Metric, symbol Device:C
- added C18: 1uF, Capacitor_SMD:C_0603_1608Metric, symbol Device:C
- added R10: 3.3k, Resistor_SMD:R_0603_1608Metric, symbol Device:R_US
- added R11: 69.8k, Resistor_SMD:R_0603_1608Metric, symbol Device:R_US
- added R13, R7, R8: 100k, Resistor_SMD:R_0603_1608Metric, symbol Device:R_US
- added R3: 43.2k, Resistor_SMD:R_0603_1608Metric, symbol Device:R_US
- added R9: 470, Resistor_SMD:R_0603_1608Metric, symbol Device:R_US
- added U4: INA819IDGK, digikey-footprints:TSSOP-8_W3mm, symbol FANTM_parts:INA819IDGK
- added U6: OPA376xxD, Package_SO:SOIC-8_3.9x4.9mm_P1.27mm, symbol Amplifier_Operational:OPA376xxD
- POT1: DK_Detail_Page https://www.digikey.com/en/products/detail/bourns-inc/TC33X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 -> /product-detail/en/bourns-inc/TC33X-2-103E/TC33X-103ETR-ND/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; Description TRIMMER 1K OHM 0.1W J LEAD TOP -> TRIMMER 10K OHM 0.1W J LEAD TOP; Digi-Key_PN TC33X-102ECT-ND -> TC33X-103ETR-ND; MPN TC33X-2-102E -> TC33X-2-103E
- R4: value 10k -> 100k; Description RES 10K OHM 1% 1/8W 0603 -> RES 100 KOHM 1% 1/10W 0603; Detailed Description 10 kOhms ±1% 0.125W, 1/8W Chip Resistor 0603 (1608 Metric) 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 -> (none); Digi-Key_PN RNCP0603FTD10K0CT-ND -> 511-1819-1-ND; MPN (none) -> SFR03EZPF1003; Manufacturer Stackpole Electronics Inc -> Rohm Semiconductor; Manufacturer Product Number RNCP0603FTD10K0 -> (none); Power (Watts) 0.125W, 1/8W -> (none); Supplier Stackpole Electronics Inc -> (none)
- R6: value 35.7k -> 1k; DK_Detail_Page https://www.digikey.com/en/products/detail/stackpole-electr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 -> (none); Description RES 35.7K OHM 1% 1/10W 0603 -> RES 1K OHM 1% 1/8W 0603; Digi-Key_PN RMCF0603FT35K7CT-ND -> RNCP0603FTD1K00CT-ND; MPN RMCF0603FT35K7 -> RNCP0603FTD1K00
- renumbered C7 to C10, C11 to C14, C12 to C15, C5 to C7, C6 to C8, R7 to R12, R1 to R2, R3 to R5, TP2 to TP4
Connections:
- net labels added: INA_N, INA_P, INA_REF, REF_-
- wire segments 88 -> 115
Other:
- note added: "AC COUPLED INSTRUMENTATION AMPLIFIER (INA)\n\nDesign referenced from \nTI's Analog Engineer's Circuit Cookbook: \nAmplifiers (Rev. A)\n\nPage 171\n"
- note added: "AC COUPLED INSTRUMENTATION AMPLIFIER (REF)\n\nDesign referenced from \nTI's Analog Engineer's Circuit Cookbook: \nAmplifiers (Rev. A)\n\nPage 171\n"
- note added: "Fc (-3dB) is 1.6Hz\nfor this high pass filter.\n"
- note added: "Fc (-3dB) is 532.5Hz\nfor this low pass filter.\n"
- note removed: "Fc (-3dB) is 611.84Hz\nfor this low pass filter.\n"
- moved on the sheet: C10, C7, C8, C9, R12, U5

Commit message: Created v1.1 of the DEVLPR, adding RLD
Parts:
- removed C11, C12: 4700pF, Capacitor_SMD:C_0603_1608Metric, symbol Device:C
- removed R10: 3.3k, Resistor_SMD:R_0603_1608Metric, symbol Device:R_US
- removed R11: 69.8k, Resistor_SMD:R_0603_1608Metric, symbol Device:R_US
- removed R3: 43.2k, Resistor_SMD:R_0603_1608Metric, symbol Device:R_US
- removed R6: 1k, Resistor_SMD:R_0603_1608Metric, symbol Device:R_US
- removed U4: INA819IDGK, digikey-footprints:TSSOP-8_W3mm, symbol FANTM_parts:INA819IDGK
- removed U5: OPA376xxD, Package_SO:SOIC-8_3.9x4.9mm_P1.27mm, symbol Amplifier_Operational:OPA376xxD
- added R?: 28.7k, symbol Device:R_US
- added R? (x2): 10k, Resistor_SMD:R_0603_1608Metric, symbol Device:R_US
- added R?: 68k, symbol Device:R_US
- added U?: OPA375DCK, digikey-footprints:SC-70-5, symbol FANTM_parts:OPA375DCK
- added U?: INA821IDGKT, digikey-footprints:TSSOP-8_W3mm, symbol FANTM_parts:INA821IDGKT
- added U?: OPA2375IPWR, Package_SO:TSSOP-8_4.4x3mm_P0.65mm, symbol FANTM_parts:OPA2375IPWR
Connections:
- net labels added: +3.3V, -3V3
- wire segments 115 -> 119
Other:
- note removed: "Fc (-3dB) is 532.5Hz\nfor this low pass filter.\n"
- moved on the sheet: R12
